File: kicad/micro-wwvb.kicad_pcb (KiCad board)
At the start: 2 copper layers, 42.5 x 40.6 mm, 20 parts, among them J2 USB_B_Mini, U1 ATtiny44A, Y1 Crystal

Commit message: Added silkscreen text to the back. Updated README.md with ATTiny info.
Other:
- board text added: "-- micro-wwvb-- Chris Genly 10/27/2023 https://github.com/chgenly/micro-wwvb.git Derived from Anish Athalye 12/18/2016 https://github.com/anishathalye/micro-wwvb.git"
- board text added: "micro-wwvb"
- board text removed: "Chris Genly micro-wwvb 10/2023"
