File: kicad/micro-wwvb.kicad_sch (KiCad schematic)
At the start: 20 parts, among them J2 USB_B_Mini, U1 ATtiny44A, Y1 Crystal

Commit message: Yikes!  I reversed all the pins on the gps connector.
I didn't realize the plug had to be turned
upside down to fit it into the connector.

The kicad files have been updated.  It also seems
I've swapped the transmit and receive on the gps
connector.  I've updated the code to compensate.
Found compatibility problems when using a windows
version of make.  Updated the makefile.
Connections:
- net GND: now also JP1.2, JP1.6; no longer JP1.1, JP1.5
- net VCC: now also JP1.5; no longer JP1.2
- no-connect marks 0 -> 1
